File: hardware/tensorrail_mini.kicad_sch (KiCad schematic)
At the start: 0 parts

Commit message: Update TensorRail schematic artifact
Parts:
- added C1, C2, C3, C4: 10uF, symbol Device:C
- added C10, C5, C6, C7, C8, C9: 100nF, symbol Device:C
- added C11: 22uF, symbol Device:C
- added J1: GCT USB4135-GF-A, symbol Custom:USB-C-GCT_USB4135-GF-A
- added J2: Feather Header Left, symbol Custom:Feather_Header
- added J3: Feather Header Right, symbol Custom:Feather_Header
- added J4: JTAG 2x5, symbol Custom:JTAG_2x5
- added J5: Expansion 2x10, symbol Custom:Expansion_2x10
- added L1, L2: 2.2uH, symbol Device:L
- added LED1: Green, symbol Device:LED
- added LED2: Blue, symbol Device:LED
- added LED3: Red, symbol Device:LED
- added R1, R2, R3, R4: 100k, symbol Device:R
- added R10: 330, symbol Device:R
- added R5, R6, R7, R8: 10k, symbol Device:R
- added R9: 0.1, symbol Device:R
- added U1, U2: TPS62130ARGTR, symbol Custom:TPS62130ARGTR
- added U3: INA219AIDCNT, symbol Custom:INA219AIDCNT
- added U4: W25Q128JVSIQ, symbol Custom:W25Q128JVSIQ
- added U5: APS6404L-3SQR, symbol Custom:APS6404L-3SQR
- added U6: CH340C, symbol Custom:CH340C
Other:
- note removed: "+1V2"
- note removed: "+3V3"
- note removed: "+5V"
- note removed: "40-pin expansion header"
- note removed: "50 MHz oscillator"
- note removed: "A0"
- note removed: "A1"
- note removed: "BOOT_N"
- note removed: "C1 10uF"
- note removed: "C13 100nF"
- note removed: "C15 100nF"
- note removed: "C2 100nF"
- note removed: "C5 100uF"
- note removed: "C6 100nF"
- note removed: "C9 100uF"
- note removed: "CC1"
- note removed: "CC2"
- note removed: "CLK"
- note removed: "CLK_50M"
- note removed: "CS#"
- note removed: "D+ NC"
- note removed: "D- NC"
- note removed: "D1 PMEG4010"
- note removed: "D3 BUSY"
- note removed: "D4 DONE"
- note removed: "D5 HEART"
- note removed: "EN"
- note removed: "FB"
- note removed: "GND"
- note removed: "GPIO"
- note removed: "HOLD#"
- note removed: "IN+"
- note removed: "IN-"
- note removed: "INA219 power monitor"
- note removed: "J1"
- note removed: "J2"
- note removed: "J3"
- note removed: "JTAG 2x5"
- note removed: "JTAG_TCK"
- note removed: "JTAG_TDI"
- note removed: "JTAG_TDO"
- note removed: "JTAG_TMS"
- note removed: "L1 2.2uH"
- note removed: "L2 1.5uH"
- note removed: "Lattice ECP5 / OrangeCrab 85F"
- note removed: "MISO"
- note removed: "MOD1"
- note removed: "MOSI"
- note removed: "OE"
- note removed: "OUT"
- note removed: "PG"
- note removed: "R1 5.1k"
- note removed: "R16 4.7k"
- note removed: "R17 4.7k"
- note removed: "R2 5.1k"
- note removed: "R3 464k"
- note removed: "R4 100k"
- note removed: "R5 103k"
- note removed: "R6 100k"
- note removed: "R7 0.1R"
- note removed: "RESET_N"
- note removed: "Reference schematic sheet: USB-C power tree, monitored ECP5 core rail, SPI boot, clock, JTAG, expansion IO."
- note removed: "SCK"
- note removed: "SCL"
- note removed: "SDA"
- note removed: "SHIELD"
- note removed: "SPI_CS"
- note removed: "SPI_MISO"
- note removed: "SPI_MOSI"
- note removed: "SPI_SCK"
- note removed: "SW"
- note removed: "SW/LED"
- note removed: "SW1 RESET"
- note removed: "SW2 BOOT"
- note removed: "TCK"
- note removed: "TDI"
- note removed: "TDO"
- note removed: "TMS"
- note removed: "TPS62130 1.2V core buck"
- note removed: "TPS62130 3.3V buck"
- note removed: "TensorRail-Mini ECP5 INT8 Accelerator Carrier"
- note removed: "U1"
- note removed: "U2"
- note removed: "U3"
- note removed: "U4"
- note removed: "U5"
- note removed: "UART_RX"
- note removed: "UART_TX"
- note removed: "USB-C power sink"
- note removed: "VBUS"
- note removed: "VCC"
- note removed: "VIN"
- note removed: "VOUT"
- note removed: "VS"
- note removed: "W25Q128 SPI flash"
- note removed: "WP#"
- note removed: "reset, boot, busy, done, heartbeat"
- company: (none) -> TensorRail
- title: (none) -> TensorRail-Mini Carrier Board

Commit message: Update TensorRail KiCad layout
Parts:
- C1, C10, C2, C3, C4, C5, C6, C7, C8, C9: footprint (none) -> Capacitor_SMD:C_0402_1005Metric
- C11: footprint (none) -> Capacitor_SMD:C_0805_2012Metric
- J1: footprint (none) -> Connector_USB:USB_C_Receptacle_GCT_USB4135
- J2, J3: footprint (none) -> Connector_PinHeader_2.54mm:PinHeader_1x16_P2.54mm_Vertical
- J4: footprint (none) -> Connector_PinHeader_2.54mm:PinHeader_2x05_P2.54mm_Vertical
- J5: footprint (none) -> Connector_PinHeader_2.54mm:PinHeader_2x10_P2.54mm_Vertical
- L1, L2: footprint (none) -> Inductor_SMD:L_Bourns-SRN4018
- LED1, LED2, LED3: footprint (none) -> LED_SMD:LED_0402_1005Metric
- R1, R10, R2, R3, R4, R5, R6, R7, R8: footprint (none) -> Resistor_SMD:R_0402_1005Metric
- R9: footprint (none) -> Resistor_SMD:R_0805_2012Metric
- U1, U2: footprint (none) -> Package_DFN_QFN:QFN-16-1EP_3x3mm_P0.5mm_EP1.45x1.45mm
- U3: footprint (none) -> Package_TO_SOT_SMD:SOT-23-8
- U4, U5: footprint (none) -> Package_SO:SOIC-8_3.9x4.9mm_P1.27mm
- U6: footprint (none) -> Package_SO:SOIC-16_3.9x9.9mm_P1.27mm
Connections:
- no-connect marks 0 -> 21

Commit message: Polish hardware signoff artifacts
Parts:
- removed C5, C6, C7, C8: 100nF, Capacitor_SMD:C_0402_1005Metric, symbol Device:C
- removed LED1: Green, LED_SMD:LED_0402_1005Metric, symbol Device:LED
- removed LED2: Blue, LED_SMD:LED_0402_1005Metric, symbol Device:LED
- removed LED3: Red, LED_SMD:LED_0402_1005Metric, symbol Device:LED
- removed R10: 330, Resistor_SMD:R_0402_1005Metric, symbol Device:R
- added D1: Green, LED_SMD:LED_0402_1005Metric, symbol Device:LED
- added D2: Yellow, LED_SMD:LED_0402_1005Metric, symbol Device:LED
- added D3: Red, LED_SMD:LED_0402_1005Metric, symbol Device:LED
- added R10, R11: 330, Resistor_SMD:R_0402_1005Metric, symbol Device:R
- added R10: 0.1, Resistor_SMD:R_2512_6332Metric, symbol Device:R
- C1, C2, C3, C4: value 10uF -> 22uF; footprint Capacitor_SMD:C_0402_1005Metric -> Capacitor_SMD:C_0805_2012Metric
- C11: value 22uF -> 100nF; footprint Capacitor_SMD:C_0805_2012Metric -> Capacitor_SMD:C_0402_1005Metric
- J2: value Feather Header Left -> Feather_Left
- J3: value Feather Header Right -> Feather_Right
- J4: value JTAG 2x5 -> JTAG_2x5; footprint Connector_PinHeader_2.54mm:PinHeader_2x05_P2.54mm_Vertical -> Connector_IDC:IDC-Header_2x05_P2.54mm_Horizontal
- J5: value Expansion 2x10 -> Expansion_2x10
- L1, L2: footprint Inductor_SMD:L_Bourns-SRN4018 -> Inductor_SMD:L_0402_1005Metric
- R2: value 100k -> 56.2k
- R3: value 100k -> 200k
- R4: value 100k -> 33.2k
- R5, R6: value 10k -> 5.1k
- R7, R8: value 10k -> 4.7k
- R9: value 0.1 -> 330; footprint Resistor_SMD:R_0805_2012Metric -> Resistor_SMD:R_0402_1005Metric
Connections:
- net +1V2: now also C4.1, L2.1, R3.1, U2.12 (BOOT), U2.13 (VOS), U3.1 (IN+), U3.2 (IN-), R10.1, R10.2
- net +3V3: now also C11.1, C2.1, C3.1, C9.1, J2.1 (Pin1), J3.1 (Pin1), J4.1 (VCC), J5.1 (P1), L1.1, L1.2, R1.1, R7.1, R8.1, R9.1, U1.10 (SW), U1.11 (SW), U1.12 (BOOT), U1.13 (VOS), U1.9 (SW), U2.1 (VIN), U2.2 (VIN), U2.3 (EN), U3.7 (VS), U4.3 (/WP), U4.7 (/HOLD), U4.8 (VCC), U5.8 (VCC), U6.16 (VCC), R10.1, R11.1
- net GND: now also C1.2, C10.2, C11.2, C2.2, C3.2, C4.2, C9.2, J1.A1/B1 (GND), J1.A12/B12 (GND), J2.16 (Pin16), J2.2 (Pin2), J3.16 (Pin16), J3.2 (Pin2), J4.3 (GND), J4.5 (GND), J4.9 (GND), J5.2 (P2), R2.2, R4.2, R5.2, R6.2, U1.17 (EPAD), U1.7 (GND), U1.8 (GND), U2.17 (EPAD), U2.7 (GND), U2.8 (GND), U3.5 (A0), U3.6 (A1), U3.8 (GND), U4.4 (GND), U5.4 (GND), U6.9 (GND), D1.2 (K), D2.2 (K), D3.2 (K)
- net SCL: now also J2.11 (Pin11), J2.12 (Pin12), R7.2, R8.2, U3.3 (SDA), U3.4 (SCL)
- net SPI_MISO: now also J2.7 (Pin7), U4.2 (DO(MISO)), U5.2 (SO/SIO1)
- net SPI_MOSI: now also J2.6 (Pin6), U4.5 (DI(MOSI)), U5.7 (SI/SIO0)
- net SPI_SCK: now also J2.5 (Pin5), U4.6 (CLK), U5.6 (SCLK)
- net VBUS_RAW: now also C1.1, J1.A4/B4 (VBUS), J1.A9/B9 (VBUS), U1.1 (VIN), U1.2 (VIN), U1.3 (EN)
- net at R4.1: now also R3.2, U2.6 (FB)
- net at R6.1: now also J1.B5 (CC2)
- net UART_RX: now reaches J2.10 (Pin10)
- net UART_RX: now also U6.3 (RXD)
- net CLK_50M: now reaches J2.13 (Pin13)
- net RESET_N: now reaches J2.3 (Pin3)
- net BOOT_N: now reaches J2.4 (Pin4)
- net FLASH_CS_N: now reaches J2.8 (Pin8)
- net FLASH_CS_N: now also U4.1 (/CS)
- net UART_TX: now reaches J2.9 (Pin9)
- net UART_TX: now also U6.2 (TXD)
- net JTAG_nRST: now reaches J4.10 (RESET)
- net JTAG_TMS: now reaches J4.2 (TMS)
- net JTAG_TCK: now reaches J4.4 (TCK)
- net JTAG_TDO: now reaches J4.6 (TDO)
- net JTAG_TDI: now reaches J4.8 (TDI)
- net at U2.10 (SW): now also L2.2, U2.11 (SW), U2.9 (SW)
- net at U1.6 (FB): now also R1.2, R2.1
- net at U6.4 (V3): now also C10.1
- net at R5.1: now also J1.A5 (CC1)
- net at R9.2: now also D1.1 (A)
- net PSRAM_CS_N: now reaches U5.1 (/CE)
- new net: D2.1 (A), R10.2
- new net: D3.1 (A), R11.2
- no-connect marks 21 -> 62
Other:
- note added: "1.2V RAIL (U2)"
- note added: "2x10 expansion header Status LEDs D1-D3 (330R) Unused pins NC"
- note added: "2x5 JTAG/SWD header JTAG_TCK/TMS/TDI/TDO/nRST"
- note added: "3.3V RAIL (U1)"
- note added: "CH340C UART bridge footprint UART_TX/RX exposed to FPGA/header domain UD+/UD- NC in this power-only USB-C revision"
- note added: "EXPANSION + LEDs (J5)"
- note added: "FLASH + PSRAM"
- note added: "FPGA MODULE (J2/J3)"
- note added: "INA219 +1V2 rail monitor 0.1 Ohm shunt → 320mA FS I2C 0x40 — SDA/SCL to FPGA"
- note added: "JTAG DEBUG (J4)"
- note added: "OrangeCrab 85F ECP5 Feather 2x16 0.1-inch pin headers (3.3V I/O)"
- note added: "POWER INPUT"
- note added: "TELEMETRY (U3)"
- note added: "UART BRIDGE (U6)"
- note added: "USB-C 5V sink only - no USB data CC1/CC2 each use 5.1k Rd to GND; D+/D-/SBU are NC"
- note added: "VIN=+3V3 VOUT=+1V2 @ 1A (FPGA core) FB: R3/R4 divider L2=2.2uH Cout=2x22uF"
- note added: "VIN=VBUS_RAW VOUT=+3V3 @ 2A FB: R1/R2 divider L1=2.2uH Cout=2x22uF"
- note added: "W25Q128 128Mb NOR flash — SPI 20MHz APS6404L 32Mb PSRAM — SPI quad-I/O"

Commit message: Align simulation artifacts with hardware design
Parts:
- L2: value 2.2uH -> 1.5uH
Other:
- note added: "VIN=+3V3 VOUT=+1V2 @ 1A (FPGA core) FB: R5/R6 divider L2=1.5uH Cout=100uF + local HF bypass"
- note removed: "VIN=+3V3 VOUT=+1V2 @ 1A (FPGA core) FB: R3/R4 divider L2=2.2uH Cout=2x22uF"
Changed lines of the file:
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@@
 		(effects (font (size 1.5 1.5) bold) (justify left))
 	)
-	(text "VIN=+3V3  VOUT=+1V2 @ 1A (FPGA core)\nFB: R3/R4 divider  L2=2.2uH  Cout=2x22uF"
+	(text "VIN=+3V3  VOUT=+1V2 @ 1A (FPGA core)\nFB: R5/R6 divider  L2=1.5uH  Cout=100uF + local HF bypass"
 		(at 89.535 62.23 0)
 		(effects (font (size 1.27 1.27)) (justify left))
@@
 			(effects (font (size 1.27 1.27)))
 		)
-		(property "Value" "2.2uH" (at 129.54 21.51 0)
-			(effects (font (size 1.27 1.27)))
-		)
+		(property "Value" "1.5uH" (at 129.54 21.51 0)
+			(effects (font (size 1.27 1.27)))
+		)
